Commit message: Fix base_link position and update RViz configuration
- Fixed base_link to be at vehicle body center (removed 0.2078m x-offset)
- Added IMU visualization plugin to RViz configuration
- Updated maintainer email in package.xml

🤖 Generated with [Claude Code](https://claude.ai/code)

Co-Authored-By: Claude <noreply@anthropic.com>

File: src/asw_robot_gazebo_sim/urdf/asw_robot_base.xacro (robot description, xacro)
@@ -45,5 +45,5 @@
         <parent link="base_link" />
         <child link="chassis_link" />
-        <origin xyz="0.2078 0.0 0.05" rpy="0 0 0" />
+        <origin xyz="0.0 0.0 0.05" rpy="0 0 0" />
     </joint>
     <!-- FRONT LEFT WHEEL -->
